Commit message: Update simulation parameters

File: scarab_description/urdf/kobuki_gazebo.urdf.xacro (robot description, xacro)
@@ -28,10 +28,10 @@
     <gazebo reference="base_link">
       <sensor type="contact" name="bumpers">
-	<always_on>1</always_on>
-	<update_rate>50.0</update_rate>
-	<visualize>true</visualize>
-	<contact>
-	  <collision>base_footprint_collision_base_link</collision>
-	</contact>
+	      <always_on>1</always_on>
+	      <update_rate>50.0</update_rate>
+	      <visualize>true</visualize>
+	      <contact>
+	        <collision>base_footprint_collision_base_link</collision>
+	      </contact>
       </sensor>
     </gazebo>
@@ -46,10 +46,15 @@
         <wheelSeparation>0.230</wheelSeparation>
         <wheelDiameter>0.070</wheelDiameter>
-        <publishWheelTF>true</publishWheelTF>
         <torque>1.0</torque>
         <commandTopic>cmd_vel</commandTopic>
-        <odometryTopic>odom_laser</odometryTopic>
-        <odometryFrame>odom_laser</odometryFrame>
-        <robotBaseFrame>base_footprint</robotBaseFrame>
+        <odometryTopic>ground_truth/odom</odometryTopic>
+        <odometryFrame>ground_truth/odom</odometryFrame>
+        <robotBaseFrame>ground_truth/base_link</robotBaseFrame>
+        <publishWheelJointState>false</publishWheelJointState>
+        <wheelAcceleration>0</wheelAcceleration>
+        <wheelTorque>5</wheelTorque>
+        <odometrySource>world</odometrySource>
+        <publishTf>1</publishTf>
+        <publishWheelTF>false</publishWheelTF>
       </plugin>
     </gazebo>

File: scarab_description/urdf/turtlebot_gazebo.urdf.xacro (robot description, xacro)
@@ -16,5 +16,5 @@
           <clip>
             <near>0.1</near>
-            <far>9.0</far>
+            <far>50.0</far>
           </clip>
         </camera>
@@ -29,5 +29,4 @@
           <depthImageCameraInfoTopicName>depth/camera_info</depthImageCameraInfoTopicName>
           <frameName>camera_depth_optical_frame</frameName>
-          <baseline>0.1</baseline>
           <distortion_k1>0.0</distortion_k1>
           <distortion_k2>0.0</distortion_k2>
@@ -36,4 +35,5 @@
           <distortion_t2>0.0</distortion_t2>
           <pointCloudCutoff>0.4</pointCloudCutoff>
+          <pointCloudCutoffMax>50.0</pointCloudCutoffMax>
         </plugin>
       </sensor>

File: scarab_description/urdf/turtlebot_properties.urdf.xacro (robot description, xacro)
@@ -19,6 +19,6 @@
      (currently in development and awaiting feedback)
    -->
-	<property name="cam_px" value="-0.087" />
-	<property name="cam_py" value="-0.0125" />
+	<property name="cam_px" value="-0.0" />
+	<property name="cam_py" value="-0.0" />
 	<property name="cam_pz" value="0.3" />
 	<property name="cam_or" value="0" />
